Commit message: corrections and some changes for a run

File: temp0.urdf (robot description, URDF)
Before this commit: robot pepe, 7 links, 6 joints
Links:
- removed link 14
- removed link 25
- removed link 26
- added link 114, mass 2.775686719147213; collision cylinder length=1.7441977173738168 radius=0.7117253431390724; visual cylinder length=1.7441977173738168 radius=0.7117253431390724
- added link 127, mass 2.775686719147213; collision cylinder length=1.7441977173738168 radius=0.7117253431390724; visual cylinder length=1.7441977173738168 radius=0.7117253431390724
- added link 215, mass 1.943957334531777; collision cylinder length=1.8640314115596583 radius=0.5761582896823306; visual cylinder length=1.8640314115596583 radius=0.5761582896823306
- added link 216, mass 1.943957334531777; collision cylinder length=1.8640314115596583 radius=0.5761582896823306; visual cylinder length=1.8640314115596583 radius=0.5761582896823306
- added link 217, mass 1.943957334531777; collision cylinder length=1.8640314115596583 radius=0.5761582896823306; visual cylinder length=1.8640314115596583 radius=0.5761582896823306
- added link 228, mass 1.943957334531777; collision cylinder length=1.8640314115596583 radius=0.5761582896823306; visual cylinder length=1.8640314115596583 radius=0.5761582896823306
- added link 229, mass 1.943957334531777; collision cylinder length=1.8640314115596583 radius=0.5761582896823306; visual cylinder length=1.8640314115596583 radius=0.5761582896823306
- added link 230, mass 1.943957334531777; collision cylinder length=1.8640314115596583 radius=0.5761582896823306; visual cylinder length=1.8640314115596583 radius=0.5761582896823306
- added link 24, mass 1.943957334531777; collision cylinder length=1.8640314115596583 radius=0.5761582896823306; visual cylinder length=1.8640314115596583 radius=0.5761582896823306
- added link 311, mass 1.3834072039895227; collision cylinder length=0.7753548623370943 radius=0.7536155008651589; visual cylinder length=0.7753548623370943 radius=0.7536155008651589
- added link 318, mass 1.3834072039895227; collision cylinder length=0.7753548623370943 radius=0.7536155008651589; visual cylinder length=0.7753548623370943 radius=0.7536155008651589
- added link 321, mass 1.3834072039895227; collision cylinder length=0.7753548623370943 radius=0.7536155008651589; visual cylinder length=0.7753548623370943 radius=0.7536155008651589
- added link 324, mass 1.3834072039895227; collision cylinder length=0.7753548623370943 radius=0.7536155008651589; visual cylinder length=0.7753548623370943 radius=0.7536155008651589
- added link 331, mass 1.3834072039895227; collision cylinder length=0.7753548623370943 radius=0.7536155008651589; visual cylinder length=0.7753548623370943 radius=0.7536155008651589
- added link 334, mass 1.3834072039895227; collision cylinder length=0.7753548623370943 radius=0.7536155008651589; visual cylinder length=0.7753548623370943 radius=0.7536155008651589
- added link 337, mass 1.3834072039895227; collision cylinder length=0.7753548623370943 radius=0.7536155008651589; visual cylinder length=0.7753548623370943 radius=0.7536155008651589
- added link 35, mass 1.3834072039895227; collision cylinder length=0.7753548623370943 radius=0.7536155008651589; visual cylinder length=0.7753548623370943 radius=0.7536155008651589
- added link 38, mass 1.3834072039895227; collision cylinder length=0.7753548623370943 radius=0.7536155008651589; visual cylinder length=0.7753548623370943 radius=0.7536155008651589
- added link 410, mass 0.18776024188554757; collision cylinder length=0.8206552117046115 radius=0.26986497087512695; visual cylinder length=0.8206552117046115 radius=0.26986497087512695
- added link 412, mass 0.18776024188554757; collision cylinder length=0.8206552117046115 radius=0.26986497087512695; visual cylinder length=0.8206552117046115 radius=0.26986497087512695
- added link 413, mass 0.18776024188554757; collision cylinder length=0.8206552117046115 radius=0.26986497087512695; visual cylinder length=0.8206552117046115 radius=0.26986497087512695
- added link 419, mass 0.18776024188554757; collision cylinder length=0.8206552117046115 radius=0.26986497087512695; visual cylinder length=0.8206552117046115 radius=0.26986497087512695
- added link 420, mass 0.18776024188554757; collision cylinder length=0.8206552117046115 radius=0.26986497087512695; visual cylinder length=0.8206552117046115 radius=0.26986497087512695
- added link 422, mass 0.18776024188554757; collision cylinder length=0.8206552117046115 radius=0.26986497087512695; visual cylinder length=0.8206552117046115 radius=0.26986497087512695
- added link 423, mass 0.18776024188554757; collision cylinder length=0.8206552117046115 radius=0.26986497087512695; visual cylinder length=0.8206552117046115 radius=0.26986497087512695
- added link 425, mass 0.18776024188554757; collision cylinder length=0.8206552117046115 radius=0.26986497087512695; visual cylinder length=0.8206552117046115 radius=0.26986497087512695
- added link 426, mass 0.18776024188554757; collision cylinder length=0.8206552117046115 radius=0.26986497087512695; visual cylinder length=0.8206552117046115 radius=0.26986497087512695
- added link 432, mass 0.18776024188554757; collision cylinder length=0.8206552117046115 radius=0.26986497087512695; visual cylinder length=0.8206552117046115 radius=0.26986497087512695
- added link 433, mass 0.18776024188554757; collision cylinder length=0.8206552117046115 radius=0.26986497087512695; visual cylinder length=0.8206552117046115 radius=0.26986497087512695
- added link 435, mass 0.18776024188554757; collision cylinder length=0.8206552117046115 radius=0.26986497087512695; visual cylinder length=0.8206552117046115 radius=0.26986497087512695
- added link 436, mass 0.18776024188554757; collision cylinder length=0.8206552117046115 radius=0.26986497087512695; visual cylinder length=0.8206552117046115 radius=0.26986497087512695
- added link 438, mass 0.18776024188554757; collision cylinder length=0.8206552117046115 radius=0.26986497087512695; visual cylinder length=0.8206552117046115 radius=0.26986497087512695
- added link 439, mass 0.18776024188554757; collision cylinder length=0.8206552117046115 radius=0.26986497087512695; visual cylinder length=0.8206552117046115 radius=0.26986497087512695
- added link 46, mass 0.18776024188554757; collision cylinder length=0.8206552117046115 radius=0.26986497087512695; visual cylinder length=0.8206552117046115 radius=0.26986497087512695
- added link 47, mass 0.18776024188554757; collision cylinder length=0.8206552117046115 radius=0.26986497087512695; visual cylinder length=0.8206552117046115 radius=0.26986497087512695
- added link 49, mass 0.18776024188554757; collision cylinder length=0.8206552117046115 radius=0.26986497087512695; visual cylinder length=0.8206552117046115 radius=0.26986497087512695
- link 0: mass 0.056087563296070564 -> 2.522596118330056; geometry collision cylinder length=1.9998 radius=0.6336590518852072; visual cylinder length=1.9998 radius=0.6336590518852072
- link 11: mass 6.281300540076709 -> 2.775686719147213; geometry collision cylinder length=1.7441977173738168 radius=0.7117253431390724; visual cylinder length=1.7441977173738168 radius=0.7117253431390724
- link 22: mass 6.281300540076709 -> 1.943957334531777; geometry collision cylinder length=1.8640314115596583 radius=0.5761582896823306; visual cylinder length=1.8640314115596583 radius=0.5761582896823306
- link 23: mass 6.281300540076709 -> 1.943957334531777; geometry collision cylinder length=1.8640314115596583 radius=0.5761582896823306; visual cylinder length=1.8640314115596583 radius=0.5761582896823306
Joints:
- removed joint 14_to_0
- removed joint 25_to_14
- removed joint 26_to_14
- added joint 114_to_0: type revolute, parent 0, child 114, origin xyz=0.7034980518682306 0.9999 0.9419078086998837 rpy=0.7608224474038389 0.16742921145481754 3.2029564512063633, axis 0 1 0, limit lower=3.1415 upper=-3.1415 effort=1 velocity=1
- added joint 127_to_0: type revolute, parent 0, child 127, origin xyz=0.7034980518682306 0.9999 0.9419078086998837 rpy=1.0144299298717852 0.16742921145481754 3.2029564512063633, axis 0 1 0, limit lower=3.1415 upper=-3.1415 effort=1 velocity=1
- added joint 215_to_114: type revolute, parent 114, child 215, origin xyz=0.03612401059642234 0.9124439586926227 0.9481717263018534 rpy=12.565113977297736 4.843686049928583 3.264299572648499, axis 0 1 0, limit lower=3.1415 upper=-3.1415 effort=1 velocity=1
- added joint 216_to_114: type revolute, parent 114, child 216, origin xyz=0.03612401059642234 0.9124439586926227 0.9481717263018534 rpy=18.847670965946605 4.843686049928583 3.264299572648499, axis 0 1 0, limit lower=3.1415 upper=-3.1415 effort=1 velocity=1
- added joint 217_to_114: type revolute, parent 114, child 217, origin xyz=0.03612401059642234 0.9124439586926227 0.9481717263018534 rpy=25.130227954595473 4.843686049928583 3.264299572648499, axis 0 1 0, limit lower=3.1415 upper=-3.1415 effort=1 velocity=1
- added joint 228_to_127: type revolute, parent 127, child 228, origin xyz=0.03612401059642234 0.9124439586926227 0.9481717263018534 rpy=12.565113977297736 4.843686049928583 3.264299572648499, axis 0 1 0, limit lower=3.1415 upper=-3.1415 effort=1 velocity=1
- added joint 229_to_127: type revolute, parent 127, child 229, origin xyz=0.03612401059642234 0.9124439586926227 0.9481717263018534 rpy=18.847670965946605 4.843686049928583 3.264299572648499, axis 0 1 0, limit lower=3.1415 upper=-3.1415 effort=1 velocity=1
- added joint 230_to_127: type revolute, parent 127, child 230, origin xyz=0.03612401059642234 0.9124439586926227 0.9481717263018534 rpy=25.130227954595473 4.843686049928583 3.264299572648499, axis 0 1 0, limit lower=3.1415 upper=-3.1415 effort=1 velocity=1
- added joint 24_to_11: type revolute, parent 11, child 24, origin xyz=0.03612401059642234 0.9124439586926227 0.9481717263018534 rpy=25.130227954595473 4.843686049928583 3.264299572648499, axis 0 1 0, limit lower=3.1415 upper=-3.1415 effort=1 velocity=1
- added joint 311_to_11: type revolute, parent 11, child 311, origin xyz=0.0 0.9999 0.27064197715547067 rpy=42.34690596106577 0.13587349341633675 6.282556988648868, axis 0 1 0, limit lower=3.1415 upper=-3.1415 effort=1 velocity=1
- added joint 318_to_114: type revolute, parent 114, child 318, origin xyz=0.0 0.9999 0.27064197715547067 rpy=30.24778997218984 0.13587349341633675 6.282556988648868, axis 0 1 0, limit lower=3.1415 upper=-3.1415 effort=1 velocity=1
- added joint 321_to_114: type revolute, parent 114, child 321, origin xyz=0.0 0.9999 0.27064197715547067 rpy=36.297347966627804 0.13587349341633675 6.282556988648868, axis 0 1 0, limit lower=3.1415 upper=-3.1415 effort=1 velocity=1
- added joint 324_to_114: type revolute, parent 114, child 324, origin xyz=0.0 0.9999 0.27064197715547067 rpy=42.34690596106577 0.13587349341633675 6.282556988648868, axis 0 1 0, limit lower=3.1415 upper=-3.1415 effort=1 velocity=1
- added joint 331_to_127: type revolute, parent 127, child 331, origin xyz=0.0 0.9999 0.27064197715547067 rpy=30.24778997218984 0.13587349341633675 6.282556988648868, axis 0 1 0, limit lower=3.1415 upper=-3.1415 effort=1 velocity=1
- added joint 334_to_127: type revolute, parent 127, child 334, origin xyz=0.0 0.9999 0.27064197715547067 rpy=36.297347966627804 0.13587349341633675 6.282556988648868, axis 0 1 0, limit lower=3.1415 upper=-3.1415 effort=1 velocity=1
- added joint 337_to_127: type revolute, parent 127, child 337, origin xyz=0.0 0.9999 0.27064197715547067 rpy=42.34690596106577 0.13587349341633675 6.282556988648868, axis 0 1 0, limit lower=3.1415 upper=-3.1415 effort=1 velocity=1
- added joint 35_to_11: type revolute, parent 11, child 35, origin xyz=0.0 0.9999 0.27064197715547067 rpy=30.24778997218984 0.13587349341633675 6.282556988648868, axis 0 1 0, limit lower=3.1415 upper=-3.1415 effort=1 velocity=1
- added joint 38_to_11: type revolute, parent 11, child 38, origin xyz=0.0 0.9999 0.27064197715547067 rpy=36.297347966627804 0.13587349341633675 6.282556988648868, axis 0 1 0, limit lower=3.1415 upper=-3.1415 effort=1 velocity=1
- added joint 410_to_38: type revolute, parent 38, child 410, origin xyz=0.6967540343136936 0.11271990472142755 0.017821480397833933 rpy=3.846105945951221 1.7654661144846993 6.118791366486142, axis 0 1 0, limit lower=3.1415 upper=-3.1415 effort=1 velocity=1
- added joint 412_to_311: type revolute, parent 311, child 412, origin xyz=0.6967540343136936 0.11271990472142755 0.017821480397833933 rpy=2.564070630634147 1.7654661144846993 6.118791366486142, axis 0 1 0, limit lower=3.1415 upper=-3.1415 effort=1 velocity=1
- added joint 413_to_311: type revolute, parent 311, child 413, origin xyz=0.6967540343136936 0.11271990472142755 0.017821480397833933 rpy=3.846105945951221 1.7654661144846993 6.118791366486142, axis 0 1 0, limit lower=3.1415 upper=-3.1415 effort=1 velocity=1
- added joint 419_to_318: type revolute, parent 318, child 419, origin xyz=0.6967540343136936 0.11271990472142755 0.017821480397833933 rpy=2.564070630634147 1.7654661144846993 6.118791366486142, axis 0 1 0, limit lower=3.1415 upper=-3.1415 effort=1 velocity=1
- added joint 420_to_318: type revolute, parent 318, child 420, origin xyz=0.6967540343136936 0.11271990472142755 0.017821480397833933 rpy=3.846105945951221 1.7654661144846993 6.118791366486142, axis 0 1 0, limit lower=3.1415 upper=-3.1415 effort=1 velocity=1
- added joint 422_to_321: type revolute, parent 321, child 422, origin xyz=0.6967540343136936 0.11271990472142755 0.017821480397833933 rpy=2.564070630634147 1.7654661144846993 6.118791366486142, axis 0 1 0, limit lower=3.1415 upper=-3.1415 effort=1 velocity=1
- added joint 423_to_321: type revolute, parent 321, child 423, origin xyz=0.6967540343136936 0.11271990472142755 0.017821480397833933 rpy=3.846105945951221 1.7654661144846993 6.118791366486142, axis 0 1 0, limit lower=3.1415 upper=-3.1415 effort=1 velocity=1
- added joint 425_to_324: type revolute, parent 324, child 425, origin xyz=0.6967540343136936 0.11271990472142755 0.017821480397833933 rpy=2.564070630634147 1.7654661144846993 6.118791366486142, axis 0 1 0, limit lower=3.1415 upper=-3.1415 effort=1 velocity=1
- added joint 426_to_324: type revolute, parent 324, child 426, origin xyz=0.6967540343136936 0.11271990472142755 0.017821480397833933 rpy=3.846105945951221 1.7654661144846993 6.118791366486142, axis 0 1 0, limit lower=3.1415 upper=-3.1415 effort=1 velocity=1
- added joint 432_to_331: type revolute, parent 331, child 432, origin xyz=0.6967540343136936 0.11271990472142755 0.017821480397833933 rpy=2.564070630634147 1.7654661144846993 6.118791366486142, axis 0 1 0, limit lower=3.1415 upper=-3.1415 effort=1 velocity=1
- added joint 433_to_331: type revolute, parent 331, child 433, origin xyz=0.6967540343136936 0.11271990472142755 0.017821480397833933 rpy=3.846105945951221 1.7654661144846993 6.118791366486142, axis 0 1 0, limit lower=3.1415 upper=-3.1415 effort=1 velocity=1
- added joint 435_to_334: type revolute, parent 334, child 435, origin xyz=0.6967540343136936 0.11271990472142755 0.017821480397833933 rpy=2.564070630634147 1.7654661144846993 6.118791366486142, axis 0 1 0, limit lower=3.1415 upper=-3.1415 effort=1 velocity=1
- added joint 436_to_334: type revolute, parent 334, child 436, origin xyz=0.6967540343136936 0.11271990472142755 0.017821480397833933 rpy=3.846105945951221 1.7654661144846993 6.118791366486142, axis 0 1 0, limit lower=3.1415 upper=-3.1415 effort=1 velocity=1
- added joint 438_to_337: type revolute, parent 337, child 438, origin xyz=0.6967540343136936 0.11271990472142755 0.017821480397833933 rpy=2.564070630634147 1.7654661144846993 6.118791366486142, axis 0 1 0, limit lower=3.1415 upper=-3.1415 effort=1 velocity=1
- added joint 439_to_337: type revolute, parent 337, child 439, origin xyz=0.6967540343136936 0.11271990472142755 0.017821480397833933 rpy=3.846105945951221 1.7654661144846993 6.118791366486142, axis 0 1 0, limit lower=3.1415 upper=-3.1415 effort=1 velocity=1
- added joint 46_to_35: type revolute, parent 35, child 46, origin xyz=0.6967540343136936 0.11271990472142755 0.017821480397833933 rpy=2.564070630634147 1.7654661144846993 6.118791366486142, axis 0 1 0, limit lower=3.1415 upper=-3.1415 effort=1 velocity=1
- added joint 47_to_35: type revolute, parent 35, child 47, origin xyz=0.6967540343136936 0.11271990472142755 0.017821480397833933 rpy=3.846105945951221 1.7654661144846993 6.118791366486142, axis 0 1 0, limit lower=3.1415 upper=-3.1415 effort=1 velocity=1
- added joint 49_to_38: type revolute, parent 38, child 49, origin xyz=0.6967540343136936 0.11271990472142755 0.017821480397833933 rpy=2.564070630634147 1.7654661144846993 6.118791366486142, axis 0 1 0, limit lower=3.1415 upper=-3.1415 effort=1 velocity=1
- joint 11_to_0: axis 0 0 1 -> 0 1 0; origin xyz=0.9999 0.9999 0.9999 rpy=12.565113977297736 6.282556988648868 6.282556988648868 -> xyz=0.7034980518682306 0.9999 0.9419078086998837 rpy=0.5072149649358926 0.16742921145481754 3.2029564512063633
- joint 22_to_11: axis 0 0 1 -> 0 1 0; origin xyz=0.9999 0.9999 0.9999 rpy=12.565113977297736 6.282556988648868 6.282556988648868 -> xyz=0.03612401059642234 0.9124439586926227 0.9481717263018534 rpy=12.565113977297736 4.843686049928583 3.264299572648499
- joint 23_to_11: axis 0 0 1 -> 0 1 0; origin xyz=0.9999 0.9999 0.9999 rpy=18.847670965946605 6.282556988648868 6.282556988648868 -> xyz=0.03612401059642234 0.9124439586926227 0.9481717263018534 rpy=18.847670965946605 4.843686049928583 3.264299572648499
