Commit message: added readme

File: temp0.urdf (robot description, URDF)
Before this commit: robot pepe, 40 links, 39 joints
Links:
- removed link 114
- removed link 127
- removed link 215
- removed link 216
- removed link 217
- removed link 228
- removed link 229
- removed link 230
- removed link 311
- removed link 318
- removed link 324
- removed link 331
- removed link 334
- removed link 38
- removed link 413
- removed link 419
- removed link 420
- removed link 425
- removed link 433
- removed link 435
- removed link 436
- removed link 49
- added link 117, mass 3.134918350295081; collision cylinder length=1.9998 radius=0.7063905792152048; visual cylinder length=1.9998 radius=0.7063905792152048
- added link 133, mass 3.134918350295081; collision cylinder length=1.9998 radius=0.7063905792152048; visual cylinder length=1.9998 radius=0.7063905792152048
- added link 218, mass 1.0253249262231574; collision cylinder length=0.3264363445720478 radius=0.9999; visual cylinder length=0.3264363445720478 radius=0.9999
- added link 219, mass 1.0253249262231574; collision cylinder length=0.3264363445720478 radius=0.9999; visual cylinder length=0.3264363445720478 radius=0.9999
- added link 220, mass 1.0253249262231574; collision cylinder length=0.3264363445720478 radius=0.9999; visual cylinder length=0.3264363445720478 radius=0.9999
- added link 234, mass 1.0253249262231574; collision cylinder length=0.3264363445720478 radius=0.9999; visual cylinder length=0.3264363445720478 radius=0.9999
- added link 235, mass 1.0253249262231574; collision cylinder length=0.3264363445720478 radius=0.9999; visual cylinder length=0.3264363445720478 radius=0.9999
- added link 236, mass 1.0253249262231574; collision cylinder length=0.3264363445720478 radius=0.9999; visual cylinder length=0.3264363445720478 radius=0.9999
- added link 313, mass 1.0858242133502927; collision cylinder length=0.34569771785372927 radius=0.9999; visual cylinder length=0.34569771785372927 radius=0.9999
- added link 325, mass 1.0858242133502927; collision cylinder length=0.34569771785372927 radius=0.9999; visual cylinder length=0.34569771785372927 radius=0.9999
- added link 329, mass 1.0858242133502927; collision cylinder length=0.34569771785372927 radius=0.9999; visual cylinder length=0.34569771785372927 radius=0.9999
- added link 341, mass 1.0858242133502927; collision cylinder length=0.34569771785372927 radius=0.9999; visual cylinder length=0.34569771785372927 radius=0.9999
- added link 345, mass 1.0858242133502927; collision cylinder length=0.34569771785372927 radius=0.9999; visual cylinder length=0.34569771785372927 radius=0.9999
- added link 39, mass 1.0858242133502927; collision cylinder length=0.34569771785372927 radius=0.9999; visual cylinder length=0.34569771785372927 radius=0.9999
- added link 411, mass 3.3463327573548867; collision cylinder length=1.1639648500576785 radius=0.9566205217931367; visual cylinder length=1.1639648500576785 radius=0.9566205217931367
- added link 414, mass 3.3463327573548867; collision cylinder length=1.1639648500576785 radius=0.9566205217931367; visual cylinder length=1.1639648500576785 radius=0.9566205217931367
- added link 415, mass 3.3463327573548867; collision cylinder length=1.1639648500576785 radius=0.9566205217931367; visual cylinder length=1.1639648500576785 radius=0.9566205217931367
- added link 416, mass 3.3463327573548867; collision cylinder length=1.1639648500576785 radius=0.9566205217931367; visual cylinder length=1.1639648500576785 radius=0.9566205217931367
- added link 424, mass 3.3463327573548867; collision cylinder length=1.1639648500576785 radius=0.9566205217931367; visual cylinder length=1.1639648500576785 radius=0.9566205217931367
- added link 427, mass 3.3463327573548867; collision cylinder length=1.1639648500576785 radius=0.9566205217931367; visual cylinder length=1.1639648500576785 radius=0.9566205217931367
- added link 428, mass 3.3463327573548867; collision cylinder length=1.1639648500576785 radius=0.9566205217931367; visual cylinder length=1.1639648500576785 radius=0.9566205217931367
- added link 430, mass 3.3463327573548867; collision cylinder length=1.1639648500576785 radius=0.9566205217931367; visual cylinder length=1.1639648500576785 radius=0.9566205217931367
- added link 431, mass 3.3463327573548867; collision cylinder length=1.1639648500576785 radius=0.9566205217931367; visual cylinder length=1.1639648500576785 radius=0.9566205217931367
- added link 440, mass 3.3463327573548867; collision cylinder length=1.1639648500576785 radius=0.9566205217931367; visual cylinder length=1.1639648500576785 radius=0.9566205217931367
- added link 442, mass 3.3463327573548867; collision cylinder length=1.1639648500576785 radius=0.9566205217931367; visual cylinder length=1.1639648500576785 radius=0.9566205217931367
- added link 443, mass 3.3463327573548867; collision cylinder length=1.1639648500576785 radius=0.9566205217931367; visual cylinder length=1.1639648500576785 radius=0.9566205217931367
- added link 444, mass 3.3463327573548867; collision cylinder length=1.1639648500576785 radius=0.9566205217931367; visual cylinder length=1.1639648500576785 radius=0.9566205217931367
- added link 446, mass 3.3463327573548867; collision cylinder length=1.1639648500576785 radius=0.9566205217931367; visual cylinder length=1.1639648500576785 radius=0.9566205217931367
- added link 447, mass 3.3463327573548867; collision cylinder length=1.1639648500576785 radius=0.9566205217931367; visual cylinder length=1.1639648500576785 radius=0.9566205217931367
- added link 448, mass 3.3463327573548867; collision cylinder length=1.1639648500576785 radius=0.9566205217931367; visual cylinder length=1.1639648500576785 radius=0.9566205217931367
- added link 48, mass 3.3463327573548867; collision cylinder length=1.1639648500576785 radius=0.9566205217931367; visual cylinder length=1.1639648500576785 radius=0.9566205217931367
- link 0: mass 2.522596118330056 -> 0.2625684372362268; geometry collision cylinder length=1.9998 radius=0.20443396002244985; visual cylinder length=1.9998 radius=0.20443396002244985
- link 11: mass 2.775686719147213 -> 3.134918350295081; geometry collision cylinder length=1.9998 radius=0.7063905792152048; visual cylinder length=1.9998 radius=0.7063905792152048
- link 22: mass 1.943957334531777 -> 1.0253249262231574; geometry collision cylinder length=0.3264363445720478 radius=0.9999; visual cylinder length=0.3264363445720478 radius=0.9999
- link 23: mass 1.943957334531777 -> 1.0253249262231574; geometry collision cylinder length=0.3264363445720478 radius=0.9999; visual cylinder length=0.3264363445720478 radius=0.9999
- link 24: mass 1.943957334531777 -> 1.0253249262231574; geometry collision cylinder length=0.3264363445720478 radius=0.9999; visual cylinder length=0.3264363445720478 radius=0.9999
- link 321: mass 1.3834072039895227 -> 1.0858242133502927; geometry collision cylinder length=0.34569771785372927 radius=0.9999; visual cylinder length=0.34569771785372927 radius=0.9999
- link 337: mass 1.3834072039895227 -> 1.0858242133502927; geometry collision cylinder length=0.34569771785372927 radius=0.9999; visual cylinder length=0.34569771785372927 radius=0.9999
- link 35: mass 1.3834072039895227 -> 1.0858242133502927; geometry collision cylinder length=0.34569771785372927 radius=0.9999; visual cylinder length=0.34569771785372927 radius=0.9999
- link 410: mass 0.18776024188554757 -> 3.3463327573548867; geometry collision cylinder length=1.1639648500576785 radius=0.9566205217931367; visual cylinder length=1.1639648500576785 radius=0.9566205217931367
- link 412: mass 0.18776024188554757 -> 3.3463327573548867; geometry collision cylinder length=1.1639648500576785 radius=0.9566205217931367; visual cylinder length=1.1639648500576785 radius=0.9566205217931367
- link 422: mass 0.18776024188554757 -> 3.3463327573548867; geometry collision cylinder length=1.1639648500576785 radius=0.9566205217931367; visual cylinder length=1.1639648500576785 radius=0.9566205217931367
- link 423: mass 0.18776024188554757 -> 3.3463327573548867; geometry collision cylinder length=1.1639648500576785 radius=0.9566205217931367; visual cylinder length=1.1639648500576785 radius=0.9566205217931367
- link 426: mass 0.18776024188554757 -> 3.3463327573548867; geometry collision cylinder length=1.1639648500576785 radius=0.9566205217931367; visual cylinder length=1.1639648500576785 radius=0.9566205217931367
- link 432: mass 0.18776024188554757 -> 3.3463327573548867; geometry collision cylinder length=1.1639648500576785 radius=0.9566205217931367; visual cylinder length=1.1639648500576785 radius=0.9566205217931367
- link 438: mass 0.18776024188554757 -> 3.3463327573548867; geometry collision cylinder length=1.1639648500576785 radius=0.9566205217931367; visual cylinder length=1.1639648500576785 radius=0.9566205217931367
- link 439: mass 0.18776024188554757 -> 3.3463327573548867; geometry collision cylinder length=1.1639648500576785 radius=0.9566205217931367; visual cylinder length=1.1639648500576785 radius=0.9566205217931367
- link 46: mass 0.18776024188554757 -> 3.3463327573548867; geometry collision cylinder length=1.1639648500576785 radius=0.9566205217931367; visual cylinder length=1.1639648500576785 radius=0.9566205217931367
- link 47: mass 0.18776024188554757 -> 3.3463327573548867; geometry collision cylinder length=1.1639648500576785 radius=0.9566205217931367; visual cylinder length=1.1639648500576785 radius=0.9566205217931367
Joints:
- removed joint 114_to_0
- removed joint 127_to_0
- removed joint 215_to_114
- removed joint 216_to_114
- removed joint 217_to_114
- removed joint 228_to_127
- removed joint 229_to_127
- removed joint 230_to_127
- removed joint 311_to_11
- removed joint 318_to_114
- removed joint 321_to_114
- removed joint 324_to_114
- removed joint 331_to_127
- removed joint 334_to_127
- removed joint 337_to_127
- removed joint 38_to_11
- removed joint 410_to_38
- removed joint 412_to_311
- removed joint 413_to_311
- removed joint 419_to_318
- removed joint 420_to_318
- removed joint 425_to_324
- removed joint 426_to_324
- removed joint 432_to_331
- removed joint 433_to_331
- removed joint 435_to_334
- removed joint 436_to_334
- removed joint 49_to_38
- added joint 117_to_0: type revolute, parent 0, child 117, origin xyz=0.03612401059642234 0.9999 0.8479822035926466 rpy=18.847670965946605 5.333198344337363 0.0, axis 0 1 0, limit lower=3.1415 upper=-3.1415 effort=1 velocity=1
- added joint 133_to_0: type revolute, parent 0, child 133, origin xyz=0.03612401059642234 0.9999 0.8479822035926466 rpy=25.130227954595473 5.333198344337363 0.0, axis 0 1 0, limit lower=3.1415 upper=-3.1415 effort=1 velocity=1
- added joint 218_to_117: type revolute, parent 117, child 218, origin xyz=0.10325470855840346 0.44354800662050825 0.3369229968491583 rpy=12.565113977297736 1.2103636104120743 0.0, axis 0 1 0, limit lower=3.1415 upper=-3.1415 effort=1 velocity=1
- added joint 219_to_117: type revolute, parent 117, child 219, origin xyz=0.10325470855840346 0.44354800662050825 0.3369229968491583 rpy=18.847670965946605 1.2103636104120743 0.0, axis 0 1 0, limit lower=3.1415 upper=-3.1415 effort=1 velocity=1
- added joint 220_to_117: type revolute, parent 117, child 220, origin xyz=0.10325470855840346 0.44354800662050825 0.3369229968491583 rpy=25.130227954595473 1.2103636104120743 0.0, axis 0 1 0, limit lower=3.1415 upper=-3.1415 effort=1 velocity=1
- added joint 234_to_133: type revolute, parent 133, child 234, origin xyz=0.10325470855840346 0.44354800662050825 0.3369229968491583 rpy=12.565113977297736 1.2103636104120743 0.0, axis 0 1 0, limit lower=3.1415 upper=-3.1415 effort=1 velocity=1
- added joint 235_to_133: type revolute, parent 133, child 235, origin xyz=0.10325470855840346 0.44354800662050825 0.3369229968491583 rpy=18.847670965946605 1.2103636104120743 0.0, axis 0 1 0, limit lower=3.1415 upper=-3.1415 effort=1 velocity=1
- added joint 236_to_133: type revolute, parent 133, child 236, origin xyz=0.10325470855840346 0.44354800662050825 0.3369229968491583 rpy=25.130227954595473 1.2103636104120743 0.0, axis 0 1 0, limit lower=3.1415 upper=-3.1415 effort=1 velocity=1
- added joint 313_to_11: type revolute, parent 11, child 313, origin xyz=0.0 0.9999 0.40576930689114155 rpy=34.127390155780425 0.0 6.282556988648868, axis 1 0 0, limit lower=3.1415 upper=-3.1415 effort=1 velocity=1
- added joint 321_to_117: type revolute, parent 117, child 321, origin xyz=0.0 0.9999 0.40576930689114155 rpy=24.376707254128874 0.0 6.282556988648868, axis 1 0 0, limit lower=3.1415 upper=-3.1415 effort=1 velocity=1
- added joint 325_to_117: type revolute, parent 117, child 325, origin xyz=0.0 0.9999 0.40576930689114155 rpy=29.252048704954646 0.0 6.282556988648868, axis 1 0 0, limit lower=3.1415 upper=-3.1415 effort=1 velocity=1
- added joint 329_to_117: type revolute, parent 117, child 329, origin xyz=0.0 0.9999 0.40576930689114155 rpy=34.127390155780425 0.0 6.282556988648868, axis 1 0 0, limit lower=3.1415 upper=-3.1415 effort=1 velocity=1
- added joint 337_to_133: type revolute, parent 133, child 337, origin xyz=0.0 0.9999 0.40576930689114155 rpy=24.376707254128874 0.0 6.282556988648868, axis 1 0 0, limit lower=3.1415 upper=-3.1415 effort=1 velocity=1
- added joint 341_to_133: type revolute, parent 133, child 341, origin xyz=0.0 0.9999 0.40576930689114155 rpy=29.252048704954646 0.0 6.282556988648868, axis 1 0 0, limit lower=3.1415 upper=-3.1415 effort=1 velocity=1
- added joint 345_to_133: type revolute, parent 133, child 345, origin xyz=0.0 0.9999 0.40576930689114155 rpy=34.127390155780425 0.0 6.282556988648868, axis 1 0 0, limit lower=3.1415 upper=-3.1415 effort=1 velocity=1
- added joint 39_to_11: type revolute, parent 11, child 39, origin xyz=0.0 0.9999 0.40576930689114155 rpy=29.252048704954646 0.0 6.282556988648868, axis 1 0 0, limit lower=3.1415 upper=-3.1415 effort=1 velocity=1
- added joint 410_to_39: type revolute, parent 39, child 410, origin xyz=0.10096680386422224 0.9999 0.7590477250910548 rpy=12.565113977297736 0.7760470795366793 5.6703595050610085, axis 1 0 0, limit lower=3.1415 upper=-3.1415 effort=1 velocity=1
- added joint 411_to_39: type revolute, parent 39, child 411, origin xyz=0.10096680386422224 0.9999 0.7590477250910548 rpy=18.847670965946605 0.7760470795366793 5.6703595050610085, axis 1 0 0, limit lower=3.1415 upper=-3.1415 effort=1 velocity=1
- added joint 412_to_39: type revolute, parent 39, child 412, origin xyz=0.10096680386422224 0.9999 0.7590477250910548 rpy=25.130227954595473 0.7760470795366793 5.6703595050610085, axis 1 0 0, limit lower=3.1415 upper=-3.1415 effort=1 velocity=1
- added joint 414_to_313: type revolute, parent 313, child 414, origin xyz=0.10096680386422224 0.9999 0.7590477250910548 rpy=12.565113977297736 0.7760470795366793 5.6703595050610085, axis 1 0 0, limit lower=3.1415 upper=-3.1415 effort=1 velocity=1
- added joint 415_to_313: type revolute, parent 313, child 415, origin xyz=0.10096680386422224 0.9999 0.7590477250910548 rpy=18.847670965946605 0.7760470795366793 5.6703595050610085, axis 1 0 0, limit lower=3.1415 upper=-3.1415 effort=1 velocity=1
- added joint 416_to_313: type revolute, parent 313, child 416, origin xyz=0.10096680386422224 0.9999 0.7590477250910548 rpy=25.130227954595473 0.7760470795366793 5.6703595050610085, axis 1 0 0, limit lower=3.1415 upper=-3.1415 effort=1 velocity=1
- added joint 424_to_321: type revolute, parent 321, child 424, origin xyz=0.10096680386422224 0.9999 0.7590477250910548 rpy=25.130227954595473 0.7760470795366793 5.6703595050610085, axis 1 0 0, limit lower=3.1415 upper=-3.1415 effort=1 velocity=1
- added joint 426_to_325: type revolute, parent 325, child 426, origin xyz=0.10096680386422224 0.9999 0.7590477250910548 rpy=12.565113977297736 0.7760470795366793 5.6703595050610085, axis 1 0 0, limit lower=3.1415 upper=-3.1415 effort=1 velocity=1
- added joint 427_to_325: type revolute, parent 325, child 427, origin xyz=0.10096680386422224 0.9999 0.7590477250910548 rpy=18.847670965946605 0.7760470795366793 5.6703595050610085, axis 1 0 0, limit lower=3.1415 upper=-3.1415 effort=1 velocity=1
- added joint 428_to_325: type revolute, parent 325, child 428, origin xyz=0.10096680386422224 0.9999 0.7590477250910548 rpy=25.130227954595473 0.7760470795366793 5.6703595050610085, axis 1 0 0, limit lower=3.1415 upper=-3.1415 effort=1 velocity=1
- added joint 430_to_329: type revolute, parent 329, child 430, origin xyz=0.10096680386422224 0.9999 0.7590477250910548 rpy=12.565113977297736 0.7760470795366793 5.6703595050610085, axis 1 0 0, limit lower=3.1415 upper=-3.1415 effort=1 velocity=1
- added joint 431_to_329: type revolute, parent 329, child 431, origin xyz=0.10096680386422224 0.9999 0.7590477250910548 rpy=18.847670965946605 0.7760470795366793 5.6703595050610085, axis 1 0 0, limit lower=3.1415 upper=-3.1415 effort=1 velocity=1
- added joint 432_to_329: type revolute, parent 329, child 432, origin xyz=0.10096680386422224 0.9999 0.7590477250910548 rpy=25.130227954595473 0.7760470795366793 5.6703595050610085, axis 1 0 0, limit lower=3.1415 upper=-3.1415 effort=1 velocity=1
- added joint 440_to_337: type revolute, parent 337, child 440, origin xyz=0.10096680386422224 0.9999 0.7590477250910548 rpy=25.130227954595473 0.7760470795366793 5.6703595050610085, axis 1 0 0, limit lower=3.1415 upper=-3.1415 effort=1 velocity=1
- added joint 442_to_341: type revolute, parent 341, child 442, origin xyz=0.10096680386422224 0.9999 0.7590477250910548 rpy=12.565113977297736 0.7760470795366793 5.6703595050610085, axis 1 0 0, limit lower=3.1415 upper=-3.1415 effort=1 velocity=1
- added joint 443_to_341: type revolute, parent 341, child 443, origin xyz=0.10096680386422224 0.9999 0.7590477250910548 rpy=18.847670965946605 0.7760470795366793 5.6703595050610085, axis 1 0 0, limit lower=3.1415 upper=-3.1415 effort=1 velocity=1
- added joint 444_to_341: type revolute, parent 341, child 444, origin xyz=0.10096680386422224 0.9999 0.7590477250910548 rpy=25.130227954595473 0.7760470795366793 5.6703595050610085, axis 1 0 0, limit lower=3.1415 upper=-3.1415 effort=1 velocity=1
- added joint 446_to_345: type revolute, parent 345, child 446, origin xyz=0.10096680386422224 0.9999 0.7590477250910548 rpy=12.565113977297736 0.7760470795366793 5.6703595050610085, axis 1 0 0, limit lower=3.1415 upper=-3.1415 effort=1 velocity=1
- added joint 447_to_345: type revolute, parent 345, child 447, origin xyz=0.10096680386422224 0.9999 0.7590477250910548 rpy=18.847670965946605 0.7760470795366793 5.6703595050610085, axis 1 0 0, limit lower=3.1415 upper=-3.1415 effort=1 velocity=1
- added joint 448_to_345: type revolute, parent 345, child 448, origin xyz=0.10096680386422224 0.9999 0.7590477250910548 rpy=25.130227954595473 0.7760470795366793 5.6703595050610085, axis 1 0 0, limit lower=3.1415 upper=-3.1415 effort=1 velocity=1
- added joint 48_to_35: type revolute, parent 35, child 48, origin xyz=0.10096680386422224 0.9999 0.7590477250910548 rpy=25.130227954595473 0.7760470795366793 5.6703595050610085, axis 1 0 0, limit lower=3.1415 upper=-3.1415 effort=1 velocity=1
- joint 11_to_0: origin xyz=0.7034980518682306 0.9999 0.9419078086998837 rpy=0.5072149649358926 0.16742921145481754 3.2029564512063633 -> xyz=0.03612401059642234 0.9999 0.8479822035926466 rpy=12.565113977297736 5.333198344337363 0.0
- joint 22_to_11: origin xyz=0.03612401059642234 0.9124439586926227 0.9481717263018534 rpy=12.565113977297736 4.843686049928583 3.264299572648499 -> xyz=0.10325470855840346 0.44354800662050825 0.3369229968491583 rpy=12.565113977297736 1.2103636104120743 0.0
- joint 23_to_11: origin xyz=0.03612401059642234 0.9124439586926227 0.9481717263018534 rpy=18.847670965946605 4.843686049928583 3.264299572648499 -> xyz=0.10325470855840346 0.44354800662050825 0.3369229968491583 rpy=18.847670965946605 1.2103636104120743 0.0
- joint 24_to_11: origin xyz=0.03612401059642234 0.9124439586926227 0.9481717263018534 rpy=25.130227954595473 4.843686049928583 3.264299572648499 -> xyz=0.10325470855840346 0.44354800662050825 0.3369229968491583 rpy=25.130227954595473 1.2103636104120743 0.0
- joint 35_to_11: axis 0 1 0 -> 1 0 0; origin xyz=0.0 0.9999 0.27064197715547067 rpy=30.24778997218984 0.13587349341633675 6.282556988648868 -> xyz=0.0 0.9999 0.40576930689114155 rpy=24.376707254128874 0.0 6.282556988648868
- joint 422_to_321: axis 0 1 0 -> 1 0 0; origin xyz=0.6967540343136936 0.11271990472142755 0.017821480397833933 rpy=2.564070630634147 1.7654661144846993 6.118791366486142 -> xyz=0.10096680386422224 0.9999 0.7590477250910548 rpy=12.565113977297736 0.7760470795366793 5.6703595050610085
- joint 423_to_321: axis 0 1 0 -> 1 0 0; origin xyz=0.6967540343136936 0.11271990472142755 0.017821480397833933 rpy=3.846105945951221 1.7654661144846993 6.118791366486142 -> xyz=0.10096680386422224 0.9999 0.7590477250910548 rpy=18.847670965946605 0.7760470795366793 5.6703595050610085
- joint 438_to_337: axis 0 1 0 -> 1 0 0; origin xyz=0.6967540343136936 0.11271990472142755 0.017821480397833933 rpy=2.564070630634147 1.7654661144846993 6.118791366486142 -> xyz=0.10096680386422224 0.9999 0.7590477250910548 rpy=12.565113977297736 0.7760470795366793 5.6703595050610085
- joint 439_to_337: axis 0 1 0 -> 1 0 0; origin xyz=0.6967540343136936 0.11271990472142755 0.017821480397833933 rpy=3.846105945951221 1.7654661144846993 6.118791366486142 -> xyz=0.10096680386422224 0.9999 0.7590477250910548 rpy=18.847670965946605 0.7760470795366793 5.6703595050610085
- joint 46_to_35: axis 0 1 0 -> 1 0 0; origin xyz=0.6967540343136936 0.11271990472142755 0.017821480397833933 rpy=2.564070630634147 1.7654661144846993 6.118791366486142 -> xyz=0.10096680386422224 0.9999 0.7590477250910548 rpy=12.565113977297736 0.7760470795366793 5.6703595050610085
- joint 47_to_35: axis 0 1 0 -> 1 0 0; origin xyz=0.6967540343136936 0.11271990472142755 0.017821480397833933 rpy=3.846105945951221 1.7654661144846993 6.118791366486142 -> xyz=0.10096680386422224 0.9999 0.7590477250910548 rpy=18.847670965946605 0.7760470795366793 5.6703595050610085
